Commit message: 새 후방 base_scan2 TF 기반 라이다 정렬,후진 및 안전 검증 적용 / URDF, bringup 설정 및 개발 테스트 모드를 기본 활성화

File: stella_description/urdf/stella.urdf (robot description, URDF)
Before this commit: robot stella, 5 links, 4 joints
Joints:
- joint scan2_joint: origin xyz=0.202 0.0 0.032 rpy=0.0 0.0 -1.57 -> xyz=-0.166 0.0 0.223 rpy=0.0 0.0 3.1415

File: stella_description/urdf/stella_web_cam.urdf (robot description, URDF)
Before this commit: robot stella, 6 links, 5 joints
Joints:
- joint scan2_joint: origin xyz=0.202 0.0 0.032 rpy=0.0 0.0 -1.57 -> xyz=-0.166 0.0 0.223 rpy=0.0 0.0 3.1415
